File: esp32tester.kicad_pcb (KiCad board)
At the start: 2 copper layers, 95 x 40.5 mm, 20 parts, among them IC1 TJA1441AT, J1 RJ45_LED_Shielded, J2 RJ45_LED_Shielded, J3 Conn_01x02_Pin, J4 Conn_01x02_Pin, J5 Screw_Terminal_01x02, J6 Conn_01x02_Pin, U1 ESP32-DevKitC

Commit message: 0518
Parts:
- moved J5 5.93 mm to (71.9, 82.2)
Routing:
- net Net-(IC1-VCC): track 95.6 -> 101.8 mm
- net GND: vias 7 -> 9
Changed lines of the file:
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@@
 		(tags "Through hole socket strip THT 1x02 2.54mm single row")
 		(property "Reference" "J4"
-			(at 2.49 1.25 0)
+			(at 2.109 1.25 0)
 			(layer "F.SilkS")
 			(effects
@@
 	(footprint "TerminalBlock_RND:TerminalBlock_RND_205-00045_1x02_P5.00mm_Horizontal"
 		(layer "F.Cu")
-		(at 77.811 82.169 180)
+		(at 71.882 82.169 180)
 		(descr "terminal block RND 205-00045, 2 pins, pitch 5mm, size 10x8.1mm^2, drill diamater 1.1mm, pad diameter 2.1mm, see http://cdn-reichelt.de/documents/datenblatt/C151/RND_205-00045_DB_EN.pdf, script-generated using https://github.com/pointhi/kicad-footprint-generator/scripts/TerminalBlock_RND")
 		(tags "THT terminal block RND 205-00045 pitch 5mm size 10x8.1mm^2 drill 1.1mm pad 2.1mm")
@@
 	)
 	(gr_text "J5"
-		(at 80.391 80.518 0)
+		(at 70.104 80.645 0)
 		(layer "B.SilkS")
 		(effects
@@
 	)
 	(gr_text "5V"
-		(at 71.755 87.757 0)
+		(at 65.913 87.63 0)
 		(layer "F.SilkS")
 		(effects
@@
 	)
 	(gr_text "GND"
-		(at 76.2 87.757 0)
+		(at 70.358 87.63 0)
 		(layer "F.SilkS")
 		(effects
@@
 	)
 	(via
+		(at 55.118 94.234)
+		(size 0.6)
+		(drill 0.3)
+		(layers "F.Cu" "B.Cu")
+		(free yes)
+		(net 1)
+	)
+	(via
 		(at 59.309 103.505)
 		(size 0.6)
@@
 		(net 1)
 	)
+	(via
+		(at 55.118 96.012)
+		(size 0.6)
+		(drill 0.3)
+		(layers "F.Cu" "B.Cu")
+		(free yes)
+		(net 1)
+	)
 	(segment
 		(start 63.393 91.009)
@@
 	)
 	(segment
-		(start 72.7975 95.9115)
-		(end 74.295 97.409)
+		(start 72.7975 90.5775)
+		(end 66.882 84.662)
 		(width 0.25)
 		(layer "F.Cu")
@@
 	)
 	(segment
-		(start 72.7975 86.2865)
-		(end 72.811 86.273)
+		(start 72.7975 95.9115)
+		(end 74.295 97.409)
 		(width 0.25)
 		(layer "F.Cu")
@@
 	)
 	(segment
-		(start 72.7975 91.948)
-		(end 72.7975 86.2865)
+		(start 72.7975 93.98)
+		(end 72.7975 95.9115)
 		(width 0.25)
 		(layer "F.Cu")
@@
 	)
 	(segment
-		(start 72.811 86.273)
-		(end 72.811 82.169)
+		(start 72.7975 91.948)
+		(end 72.7975 90.5775)
 		(width 0.25)
 		(layer "F.Cu")
@@
 	)
 	(segment
-		(start 72.7975 93.98)
-		(end 72.7975 95.9115)
+		(start 72.7975 91.948)
+		(end 72.7975 93.98)
 		(width 0.25)
 		(layer "F.Cu")
@@
 	)
 	(segment
-		(start 72.7975 91.948)
-		(end 72.7975 93.98)
+		(start 66.882 84.662)
+		(end 66.882 82.169)
 		(width 0.25)
 		(layer "F.Cu")
@@
 	)
 	(segment
-		(start 72.811 85.8628)
-		(end 72.811 82.169)
+		(start 129.55016 111.0234)
+		(end 129.55016 106.61396)
 		(width 1)
 		(layer "B.Cu")
@@
 	)
 	(segment
-		(start 85.6996 98.8314)
-		(end 72.771 85.9028)
-		(width 1)
-		(layer "B.Cu")
-		(net 4)
-	)
-	(segment
-		(start 129.55016 111.0234)
-		(end 129.55016 106.61396)
-		(width 1)
-		(layer "B.Cu")
-		(net 4)
-	)
-	(segment
-		(start 72.771 85.9028)
-		(end 72.811 85.8628)
+		(start 129.55016 106.61396)
+		(end 121.7676 98.8314)
 		(width 1)
 		(layer "B.Cu")
@@
 	)
 	(segment
-		(start 129.55016 106.61396)
-		(end 121.7676 98.8314)
+		(start 83.5444 98.8314)
+		(end 66.882 82.169)
 		(width 1)
 		(layer "B.Cu")
@@
 	(segment
 		(start 121.7676 98.8314)
-		(end 85.6996 98.8314)
+		(end 83.5444 98.8314)
 		(width 1)
 		(layer "B.Cu")
